Commit message: create custom 40ft

File: custom5ftstraight.urdf (robot description, URDF)
Before this commit: robot roller_conveyor, 17 links, 16 joints
Links:
- link base_link: geometry collision box size=1.65 1.219 0.1; visual box size=1.65 1.219 0.1
- link leftFrame: geometry collision box size=1.65 0.05 0.5; visual box size=1.65 0.05 0.5
- link rightFrame: geometry collision box size=1.65 0.05 0.5; visual box size=1.65 0.05 0.5
Joints:
- joint roller_10_joint: mimic (none) -> joint=roller_1_joint multiplier=1.0
- joint roller_11_joint: mimic (none) -> joint=roller_1_joint multiplier=1.0
- joint roller_12_joint: mimic (none) -> joint=roller_1_joint multiplier=1.0
- joint roller_13_joint: mimic (none) -> joint=roller_1_joint multiplier=1.0
- joint roller_14_joint: mimic (none) -> joint=roller_1_joint multiplier=1.0
- joint roller_1_joint: limit (none) -> lower=-180.0 upper=180.0 effort=0.0 velocity=10.0
- joint roller_2_joint: mimic (none) -> joint=roller_1_joint multiplier=1.0
- joint roller_3_joint: mimic (none) -> joint=roller_1_joint multiplier=1.0
- joint roller_4_joint: mimic (none) -> joint=roller_1_joint multiplier=1.0
- joint roller_5_joint: mimic (none) -> joint=roller_1_joint multiplier=1.0
- joint roller_6_joint: mimic (none) -> joint=roller_1_joint multiplier=1.0
- joint roller_7_joint: mimic (none) -> joint=roller_1_joint multiplier=1.0
- joint roller_8_joint: mimic (none) -> joint=roller_1_joint multiplier=1.0
- joint roller_9_joint: mimic (none) -> joint=roller_1_joint multiplier=1.0
