Commit message: change back to continuous

File: custom40ftStraight.urdf (robot description, URDF)
Before this commit: robot roller_conveyor_40ft, 131 links, 130 joints
Joints:
- joint Roller_1_joint: limit lower=-10.0 upper=10.0 effort=0.0 velocity=10.0 -> (none); type revolute -> continuous
- joint Roller_33_joint: limit lower=-10.0 upper=10.0 effort=0.0 velocity=10.0 -> (none); type revolute -> continuous
- joint Roller_65_joint: limit lower=-10.0 upper=10.0 effort=0.0 velocity=10.0 -> (none); type revolute -> continuous
- joint Roller_97_joint: limit lower=-10.0 upper=10.0 effort=0.0 velocity=10.0 -> (none); type revolute -> continuous

File: custom40ftStraight.xacro (robot description, xacro)
@@ -113,10 +113,9 @@
         </inertial>
     </link>
-    <joint name="Roller_1_joint" type="revolute">
+    <joint name="Roller_1_joint" type="continuous">
         <parent link="base_link"/>
         <child link="Roller_1"/>
         <origin xyz="-${roller_pitch/2} 0 0.15" rpy="1.570796 0 0"/>
         <axis xyz="0 0 1"/>
-        <limit lower="-10.0" upper="10.0" effort="0.0" velocity="10.0"/>
         <dynamics damping="0.1" friction="0.2"/>
     </joint>
@@ -172,10 +171,9 @@
         </inertial>
     </link>
-    <joint name="Roller_33_joint" type="revolute">
+    <joint name="Roller_33_joint" type="continuous">
         <parent link="base_link"/>
         <child link="Roller_33"/>
         <origin xyz="-${(32)*roller_pitch + roller_pitch/2} 0 0.15" rpy="1.570796 0 0"/>
         <axis xyz="0 0 1"/>
-        <limit lower="-10.0" upper="10.0" effort="0.0" velocity="10.0"/>
         <dynamics damping="0.1" friction="0.2"/>
     </joint>
@@ -231,10 +229,9 @@
         </inertial>
     </link>
-    <joint name="Roller_65_joint" type="revolute">
+    <joint name="Roller_65_joint" type="continuous">
         <parent link="base_link"/>
         <child link="Roller_65"/>
         <origin xyz="-${(64)*roller_pitch + roller_pitch/2} 0 0.15" rpy="1.570796 0 0"/>
         <axis xyz="0 0 1"/>
-        <limit lower="-10.0" upper="10.0" effort="0.0" velocity="10.0"/>
         <dynamics damping="0.1" friction="0.2"/>
     </joint>
@@ -290,10 +287,9 @@
         </inertial>
     </link>
-    <joint name="Roller_97_joint" type="revolute">
+    <joint name="Roller_97_joint" type="continuous">
         <parent link="base_link"/>
         <child link="Roller_97"/>
         <origin xyz="-${(96)*roller_pitch + roller_pitch/2} 0 0.15" rpy="1.570796 0 0"/>
         <axis xyz="0 0 1"/>
-        <limit lower="-10.0" upper="10.0" effort="0.0" velocity="10.0"/>
         <dynamics damping="0.1" friction="0.2"/>
     </joint>

Commit message: Finished CreateFCEnv.py

File: custom40ftStraight.urdf (robot description, URDF)
Before this commit: robot roller_conveyor_40ft, 131 links, 130 joints
Joints:
- joint Roller_2_joint: origin xyz=-0.142875 0 0.15 rpy=1.5707963 0 0 -> xyz=-0.142875 0 0.15 rpy=1.570796 0 0
