Commit message: new urdf

File: custom40ftStraight.urdf (robot description, URDF)
Before this commit: robot roller_conveyor_40ft, 131 links, 130 joints
Joints:
- removed joint Roller_100_joint
- removed joint Roller_101_joint
- removed joint Roller_102_joint
- removed joint Roller_103_joint
- removed joint Roller_104_joint
- removed joint Roller_105_joint
- removed joint Roller_106_joint
- removed joint Roller_107_joint
- removed joint Roller_108_joint
- removed joint Roller_109_joint
- removed joint Roller_10_joint
- removed joint Roller_110_joint
- removed joint Roller_111_joint
- removed joint Roller_112_joint
- removed joint Roller_113_joint
- removed joint Roller_114_joint
- removed joint Roller_115_joint
- removed joint Roller_116_joint
- removed joint Roller_117_joint
- removed joint Roller_118_joint
- removed joint Roller_119_joint
- removed joint Roller_11_joint
- removed joint Roller_120_joint
- removed joint Roller_121_joint
- removed joint Roller_122_joint
- removed joint Roller_123_joint
- removed joint Roller_124_joint
- removed joint Roller_125_joint
- removed joint Roller_126_joint
- removed joint Roller_127_joint
- removed joint Roller_128_joint
- removed joint Roller_12_joint
- removed joint Roller_13_joint
- removed joint Roller_14_joint
- removed joint Roller_15_joint
- removed joint Roller_16_joint
- removed joint Roller_17_joint
- removed joint Roller_18_joint
- removed joint Roller_19_joint
- removed joint Roller_1_joint
- removed joint Roller_20_joint
- removed joint Roller_21_joint
- removed joint Roller_22_joint
- removed joint Roller_23_joint
- removed joint Roller_24_joint
- removed joint Roller_25_joint
- removed joint Roller_26_joint
- removed joint Roller_27_joint
- removed joint Roller_28_joint
- removed joint Roller_29_joint
- removed joint Roller_2_joint
- removed joint Roller_30_joint
- removed joint Roller_31_joint
- removed joint Roller_32_joint
- removed joint Roller_33_joint
- removed joint Roller_34_joint
- removed joint Roller_35_joint
- removed joint Roller_36_joint
- removed joint Roller_37_joint
- removed joint Roller_38_joint
- removed joint Roller_39_joint
- removed joint Roller_3_joint
- removed joint Roller_40_joint
- removed joint Roller_41_joint
- removed joint Roller_42_joint
- removed joint Roller_43_joint
- removed joint Roller_44_joint
- removed joint Roller_45_joint
- removed joint Roller_46_joint
- removed joint Roller_47_joint
- removed joint Roller_48_joint
- removed joint Roller_49_joint
- removed joint Roller_4_joint
- removed joint Roller_50_joint
- removed joint Roller_51_joint
- removed joint Roller_52_joint
- removed joint Roller_53_joint
- removed joint Roller_54_joint
- removed joint Roller_55_joint
- removed joint Roller_56_joint
- removed joint Roller_57_joint
- removed joint Roller_58_joint
- removed joint Roller_59_joint
- removed joint Roller_5_joint
- removed joint Roller_60_joint
- removed joint Roller_61_joint
- removed joint Roller_62_joint
- removed joint Roller_63_joint
- removed joint Roller_64_joint
- removed joint Roller_65_joint
- removed joint Roller_66_joint
- removed joint Roller_67_joint
- removed joint Roller_68_joint
- removed joint Roller_69_joint
- removed joint Roller_6_joint
- removed joint Roller_70_joint
- removed joint Roller_71_joint
- removed joint Roller_72_joint
- removed joint Roller_73_joint
- removed joint Roller_74_joint
- removed joint Roller_75_joint
- removed joint Roller_76_joint
- removed joint Roller_77_joint
- removed joint Roller_78_joint
- removed joint Roller_79_joint
- removed joint Roller_7_joint
- removed joint Roller_80_joint
- removed joint Roller_81_joint
- removed joint Roller_82_joint
- removed joint Roller_83_joint
- removed joint Roller_84_joint
- removed joint Roller_85_joint
- removed joint Roller_86_joint
- removed joint Roller_87_joint
- removed joint Roller_88_joint
- removed joint Roller_89_joint
- removed joint Roller_8_joint
- removed joint Roller_90_joint
- removed joint Roller_91_joint
- removed joint Roller_92_joint
- removed joint Roller_93_joint
- removed joint Roller_94_joint
- removed joint Roller_95_joint
- removed joint Roller_96_joint
- removed joint Roller_97_joint
- removed joint Roller_98_joint
- removed joint Roller_99_joint
- removed joint Roller_9_joint
- added joint Roller_1_10_joint: type continuous, parent base_link, child Roller_10, origin xyz=-0.9048750000000001 0 0.15 rpy=1.5707963 0 0, axis 0 0 1
- added joint Roller_1_11_joint: type continuous, parent base_link, child Roller_11, origin xyz=-1.000125 0 0.15 rpy=1.5707963 0 0, axis 0 0 1
- added joint Roller_1_12_joint: type continuous, parent base_link, child Roller_12, origin xyz=-1.095375 0 0.15 rpy=1.5707963 0 0, axis 0 0 1
- added joint Roller_1_13_joint: type continuous, parent base_link, child Roller_13, origin xyz=-1.190625 0 0.15 rpy=1.5707963 0 0, axis 0 0 1
- added joint Roller_1_14_joint: type continuous, parent base_link, child Roller_14, origin xyz=-1.285875 0 0.15 rpy=1.5707963 0 0, axis 0 0 1
- added joint Roller_1_15_joint: type continuous, parent base_link, child Roller_15, origin xyz=-1.381125 0 0.15 rpy=1.5707963 0 0, axis 0 0 1
- added joint Roller_1_16_joint: type continuous, parent base_link, child Roller_16, origin xyz=-1.476375 0 0.15 rpy=1.5707963 0 0, axis 0 0 1
- added joint Roller_1_17_joint: type continuous, parent base_link, child Roller_17, origin xyz=-1.571625 0 0.15 rpy=1.5707963 0 0, axis 0 0 1
- added joint Roller_1_18_joint: type continuous, parent base_link, child Roller_18, origin xyz=-1.666875 0 0.15 rpy=1.5707963 0 0, axis 0 0 1
- added joint Roller_1_19_joint: type continuous, parent base_link, child Roller_19, origin xyz=-1.7621250000000002 0 0.15 rpy=1.5707963 0 0, axis 0 0 1
- added joint Roller_1_1_joint: type continuous, parent base_link, child Roller_1, origin xyz=-0.047625 0 0.15 rpy=1.570796 0 0, axis 0 0 1
- added joint Roller_1_20_joint: type continuous, parent base_link, child Roller_20, origin xyz=-1.857375 0 0.15 rpy=1.5707963 0 0, axis 0 0 1
- added joint Roller_1_21_joint: type continuous, parent base_link, child Roller_21, origin xyz=-1.952625 0 0.15 rpy=1.5707963 0 0, axis 0 0 1
- added joint Roller_1_22_joint: type continuous, parent base_link, child Roller_22, origin xyz=-2.047875 0 0.15 rpy=1.5707963 0 0, axis 0 0 1
- added joint Roller_1_23_joint: type continuous, parent base_link, child Roller_23, origin xyz=-2.143125 0 0.15 rpy=1.5707963 0 0, axis 0 0 1
- added joint Roller_1_24_joint: type continuous, parent base_link, child Roller_24, origin xyz=-2.238375 0 0.15 rpy=1.5707963 0 0, axis 0 0 1
- added joint Roller_1_25_joint: type continuous, parent base_link, child Roller_25, origin xyz=-2.333625 0 0.15 rpy=1.5707963 0 0, axis 0 0 1
- added joint Roller_1_26_joint: type continuous, parent base_link, child Roller_26, origin xyz=-2.428875 0 0.15 rpy=1.5707963 0 0, axis 0 0 1
- added joint Roller_1_27_joint: type continuous, parent base_link, child Roller_27, origin xyz=-2.524125 0 0.15 rpy=1.5707963 0 0, axis 0 0 1
- added joint Roller_1_28_joint: type continuous, parent base_link, child Roller_28, origin xyz=-2.6193750000000002 0 0.15 rpy=1.5707963 0 0, axis 0 0 1
- added joint Roller_1_29_joint: type continuous, parent base_link, child Roller_29, origin xyz=-2.714625 0 0.15 rpy=1.5707963 0 0, axis 0 0 1
- added joint Roller_1_2_joint: type continuous, parent base_link, child Roller_2, origin xyz=-0.142875 0 0.15 rpy=1.5707963 0 0, axis 0 0 1
- added joint Roller_1_30_joint: type continuous, parent base_link, child Roller_30, origin xyz=-2.809875 0 0.15 rpy=1.5707963 0 0, axis 0 0 1
- added joint Roller_1_31_joint: type continuous, parent base_link, child Roller_31, origin xyz=-2.905125 0 0.15 rpy=1.5707963 0 0, axis 0 0 1
- added joint Roller_1_32_joint: type continuous, parent base_link, child Roller_32, origin xyz=-3.000375 0 0.15 rpy=1.5707963 0 0, axis 0 0 1
- added joint Roller_1_3_joint: type continuous, parent base_link, child Roller_3, origin xyz=-0.238125 0 0.15 rpy=1.5707963 0 0, axis 0 0 1
- added joint Roller_1_4_joint: type continuous, parent base_link, child Roller_4, origin xyz=-0.333375 0 0.15 rpy=1.5707963 0 0, axis 0 0 1
- added joint Roller_1_5_joint: type continuous, parent base_link, child Roller_5, origin xyz=-0.42862500000000003 0 0.15 rpy=1.5707963 0 0, axis 0 0 1
- added joint Roller_1_6_joint: type continuous, parent base_link, child Roller_6, origin xyz=-0.523875 0 0.15 rpy=1.5707963 0 0, axis 0 0 1
- added joint Roller_1_7_joint: type continuous, parent base_link, child Roller_7, origin xyz=-0.619125 0 0.15 rpy=1.5707963 0 0, axis 0 0 1
- added joint Roller_1_8_joint: type continuous, parent base_link, child Roller_8, origin xyz=-0.714375 0 0.15 rpy=1.5707963 0 0, axis 0 0 1
- added joint Roller_1_9_joint: type continuous, parent base_link, child Roller_9, origin xyz=-0.809625 0 0.15 rpy=1.5707963 0 0, axis 0 0 1
- added joint Roller_33_33_joint: type continuous, parent base_link, child Roller_33, origin xyz=-3.095625 0 0.15 rpy=1.570796 0 0, axis 0 0 1
- added joint Roller_33_34_joint: type continuous, parent base_link, child Roller_34, origin xyz=-3.190875 0 0.15 rpy=1.5707963 0 0, axis 0 0 1
- added joint Roller_33_35_joint: type continuous, parent base_link, child Roller_35, origin xyz=-3.286125 0 0.15 rpy=1.5707963 0 0, axis 0 0 1
- added joint Roller_33_36_joint: type continuous, parent base_link, child Roller_36, origin xyz=-3.3813750000000002 0 0.15 rpy=1.5707963 0 0, axis 0 0 1
- added joint Roller_33_37_joint: type continuous, parent base_link, child Roller_37, origin xyz=-3.4766250000000003 0 0.15 rpy=1.5707963 0 0, axis 0 0 1
- added joint Roller_33_38_joint: type continuous, parent base_link, child Roller_38, origin xyz=-3.571875 0 0.15 rpy=1.5707963 0 0, axis 0 0 1
- added joint Roller_33_39_joint: type continuous, parent base_link, child Roller_39, origin xyz=-3.667125 0 0.15 rpy=1.5707963 0 0, axis 0 0 1
- added joint Roller_33_40_joint: type continuous, parent base_link, child Roller_40, origin xyz=-3.762375 0 0.15 rpy=1.5707963 0 0, axis 0 0 1
- added joint Roller_33_41_joint: type continuous, parent base_link, child Roller_41, origin xyz=-3.857625 0 0.15 rpy=1.5707963 0 0, axis 0 0 1
- added joint Roller_33_42_joint: type continuous, parent base_link, child Roller_42, origin xyz=-3.952875 0 0.15 rpy=1.5707963 0 0, axis 0 0 1
- added joint Roller_33_43_joint: type continuous, parent base_link, child Roller_43, origin xyz=-4.048125 0 0.15 rpy=1.5707963 0 0, axis 0 0 1
- added joint Roller_33_44_joint: type continuous, parent base_link, child Roller_44, origin xyz=-4.143375 0 0.15 rpy=1.5707963 0 0, axis 0 0 1
- added joint Roller_33_45_joint: type continuous, parent base_link, child Roller_45, origin xyz=-4.238625 0 0.15 rpy=1.5707963 0 0, axis 0 0 1
- added joint Roller_33_46_joint: type continuous, parent base_link, child Roller_46, origin xyz=-4.333875 0 0.15 rpy=1.5707963 0 0, axis 0 0 1
- added joint Roller_33_47_joint: type continuous, parent base_link, child Roller_47, origin xyz=-4.429125 0 0.15 rpy=1.5707963 0 0, axis 0 0 1
- added joint Roller_33_48_joint: type continuous, parent base_link, child Roller_48, origin xyz=-4.524375 0 0.15 rpy=1.5707963 0 0, axis 0 0 1
- added joint Roller_33_49_joint: type continuous, parent base_link, child Roller_49, origin xyz=-4.619625 0 0.15 rpy=1.5707963 0 0, axis 0 0 1
- added joint Roller_33_50_joint: type continuous, parent base_link, child Roller_50, origin xyz=-4.714875 0 0.15 rpy=1.5707963 0 0, axis 0 0 1
- added joint Roller_33_51_joint: type continuous, parent base_link, child Roller_51, origin xyz=-4.810125 0 0.15 rpy=1.5707963 0 0, axis 0 0 1
- added joint Roller_33_52_joint: type continuous, parent base_link, child Roller_52, origin xyz=-4.905375 0 0.15 rpy=1.5707963 0 0, axis 0 0 1
- added joint Roller_33_53_joint: type continuous, parent base_link, child Roller_53, origin xyz=-5.000625 0 0.15 rpy=1.5707963 0 0, axis 0 0 1
- added joint Roller_33_54_joint: type continuous, parent base_link, child Roller_54, origin xyz=-5.095875 0 0.15 rpy=1.5707963 0 0, axis 0 0 1
- added joint Roller_33_55_joint: type continuous, parent base_link, child Roller_55, origin xyz=-5.191125 0 0.15 rpy=1.5707963 0 0, axis 0 0 1
- added joint Roller_33_56_joint: type continuous, parent base_link, child Roller_56, origin xyz=-5.2863750000000005 0 0.15 rpy=1.5707963 0 0, axis 0 0 1
- added joint Roller_33_57_joint: type continuous, parent base_link, child Roller_57, origin xyz=-5.381625 0 0.15 rpy=1.5707963 0 0, axis 0 0 1
- added joint Roller_33_58_joint: type continuous, parent base_link, child Roller_58, origin xyz=-5.476875 0 0.15 rpy=1.5707963 0 0, axis 0 0 1
- added joint Roller_33_59_joint: type continuous, parent base_link, child Roller_59, origin xyz=-5.572125 0 0.15 rpy=1.5707963 0 0, axis 0 0 1
- added joint Roller_33_60_joint: type continuous, parent base_link, child Roller_60, origin xyz=-5.667375 0 0.15 rpy=1.5707963 0 0, axis 0 0 1
- added joint Roller_33_61_joint: type continuous, parent base_link, child Roller_61, origin xyz=-5.762625 0 0.15 rpy=1.5707963 0 0, axis 0 0 1
- added joint Roller_33_62_joint: type continuous, parent base_link, child Roller_62, origin xyz=-5.857875 0 0.15 rpy=1.5707963 0 0, axis 0 0 1
- added joint Roller_33_63_joint: type continuous, parent base_link, child Roller_63, origin xyz=-5.953125 0 0.15 rpy=1.5707963 0 0, axis 0 0 1
- added joint Roller_33_64_joint: type continuous, parent base_link, child Roller_64, origin xyz=-6.048375 0 0.15 rpy=1.5707963 0 0, axis 0 0 1
- added joint Roller_65_65_joint: type continuous, parent base_link, child Roller_65, origin xyz=-6.143625 0 0.15 rpy=1.570796 0 0, axis 0 0 1
- added joint Roller_65_66_joint: type continuous, parent base_link, child Roller_66, origin xyz=-6.238875 0 0.15 rpy=1.5707963 0 0, axis 0 0 1
- added joint Roller_65_67_joint: type continuous, parent base_link, child Roller_67, origin xyz=-6.334125 0 0.15 rpy=1.5707963 0 0, axis 0 0 1
- added joint Roller_65_68_joint: type continuous, parent base_link, child Roller_68, origin xyz=-6.429375 0 0.15 rpy=1.5707963 0 0, axis 0 0 1
- added joint Roller_65_69_joint: type continuous, parent base_link, child Roller_69, origin xyz=-6.524625 0 0.15 rpy=1.5707963 0 0, axis 0 0 1
- added joint Roller_65_70_joint: type continuous, parent base_link, child Roller_70, origin xyz=-6.619875 0 0.15 rpy=1.5707963 0 0, axis 0 0 1
- added joint Roller_65_71_joint: type continuous, parent base_link, child Roller_71, origin xyz=-6.7151250000000005 0 0.15 rpy=1.5707963 0 0, axis 0 0 1
- added joint Roller_65_72_joint: type continuous, parent base_link, child Roller_72, origin xyz=-6.8103750000000005 0 0.15 rpy=1.5707963 0 0, axis 0 0 1
- added joint Roller_65_73_joint: type continuous, parent base_link, child Roller_73, origin xyz=-6.905625000000001 0 0.15 rpy=1.5707963 0 0, axis 0 0 1
- added joint Roller_65_74_joint: type continuous, parent base_link, child Roller_74, origin xyz=-7.000875 0 0.15 rpy=1.5707963 0 0, axis 0 0 1
- added joint Roller_65_75_joint: type continuous, parent base_link, child Roller_75, origin xyz=-7.096125 0 0.15 rpy=1.5707963 0 0, axis 0 0 1
- added joint Roller_65_76_joint: type continuous, parent base_link, child Roller_76, origin xyz=-7.191375 0 0.15 rpy=1.5707963 0 0, axis 0 0 1
- added joint Roller_65_77_joint: type continuous, parent base_link, child Roller_77, origin xyz=-7.286625 0 0.15 rpy=1.5707963 0 0, axis 0 0 1
- added joint Roller_65_78_joint: type continuous, parent base_link, child Roller_78, origin xyz=-7.381875 0 0.15 rpy=1.5707963 0 0, axis 0 0 1
- added joint Roller_65_79_joint: type continuous, parent base_link, child Roller_79, origin xyz=-7.477125 0 0.15 rpy=1.5707963 0 0, axis 0 0 1
- added joint Roller_65_80_joint: type continuous, parent base_link, child Roller_80, origin xyz=-7.572375 0 0.15 rpy=1.5707963 0 0, axis 0 0 1
- added joint Roller_65_81_joint: type continuous, parent base_link, child Roller_81, origin xyz=-7.667625 0 0.15 rpy=1.5707963 0 0, axis 0 0 1
- added joint Roller_65_82_joint: type continuous, parent base_link, child Roller_82, origin xyz=-7.762875 0 0.15 rpy=1.5707963 0 0, axis 0 0 1
- added joint Roller_65_83_joint: type continuous, parent base_link, child Roller_83, origin xyz=-7.858125 0 0.15 rpy=1.5707963 0 0, axis 0 0 1
- added joint Roller_65_84_joint: type continuous, parent base_link, child Roller_84, origin xyz=-7.953375 0 0.15 rpy=1.5707963 0 0, axis 0 0 1
- added joint Roller_65_85_joint: type continuous, parent base_link, child Roller_85, origin xyz=-8.048625 0 0.15 rpy=1.5707963 0 0, axis 0 0 1
- added joint Roller_65_86_joint: type continuous, parent base_link, child Roller_86, origin xyz=-8.143875 0 0.15 rpy=1.5707963 0 0, axis 0 0 1
- added joint Roller_65_87_joint: type continuous, parent base_link, child Roller_87, origin xyz=-8.239125 0 0.15 rpy=1.5707963 0 0, axis 0 0 1
- added joint Roller_65_88_joint: type continuous, parent base_link, child Roller_88, origin xyz=-8.334375 0 0.15 rpy=1.5707963 0 0, axis 0 0 1
- added joint Roller_65_89_joint: type continuous, parent base_link, child Roller_89, origin xyz=-8.429625 0 0.15 rpy=1.5707963 0 0, axis 0 0 1
- added joint Roller_65_90_joint: type continuous, parent base_link, child Roller_90, origin xyz=-8.524875 0 0.15 rpy=1.5707963 0 0, axis 0 0 1
- added joint Roller_65_91_joint: type continuous, parent base_link, child Roller_91, origin xyz=-8.620125 0 0.15 rpy=1.5707963 0 0, axis 0 0 1
- added joint Roller_65_92_joint: type continuous, parent base_link, child Roller_92, origin xyz=-8.715375 0 0.15 rpy=1.5707963 0 0, axis 0 0 1
- added joint Roller_65_93_joint: type continuous, parent base_link, child Roller_93, origin xyz=-8.810625 0 0.15 rpy=1.5707963 0 0, axis 0 0 1
- added joint Roller_65_94_joint: type continuous, parent base_link, child Roller_94, origin xyz=-8.905875 0 0.15 rpy=1.5707963 0 0, axis 0 0 1
- added joint Roller_65_95_joint: type continuous, parent base_link, child Roller_95, origin xyz=-9.001125 0 0.15 rpy=1.5707963 0 0, axis 0 0 1
- added joint Roller_65_96_joint: type continuous, parent base_link, child Roller_96, origin xyz=-9.096375 0 0.15 rpy=1.5707963 0 0, axis 0 0 1
- added joint Roller_97_100_joint: type continuous, parent base_link, child Roller_100, origin xyz=-9.477375 0 0.15 rpy=1.5707963 0 0, axis 0 0 1
- added joint Roller_97_101_joint: type continuous, parent base_link, child Roller_101, origin xyz=-9.572625 0 0.15 rpy=1.5707963 0 0, axis 0 0 1
- added joint Roller_97_102_joint: type continuous, parent base_link, child Roller_102, origin xyz=-9.667875 0 0.15 rpy=1.5707963 0 0, axis 0 0 1
- added joint Roller_97_103_joint: type continuous, parent base_link, child Roller_103, origin xyz=-9.763125 0 0.15 rpy=1.5707963 0 0, axis 0 0 1
- added joint Roller_97_104_joint: type continuous, parent base_link, child Roller_104, origin xyz=-9.858375 0 0.15 rpy=1.5707963 0 0, axis 0 0 1
- added joint Roller_97_105_joint: type continuous, parent base_link, child Roller_105, origin xyz=-9.953625 0 0.15 rpy=1.5707963 0 0, axis 0 0 1
- added joint Roller_97_106_joint: type continuous, parent base_link, child Roller_106, origin xyz=-10.048875 0 0.15 rpy=1.5707963 0 0, axis 0 0 1
- added joint Roller_97_107_joint: type continuous, parent base_link, child Roller_107, origin xyz=-10.144125 0 0.15 rpy=1.5707963 0 0, axis 0 0 1
- added joint Roller_97_108_joint: type continuous, parent base_link, child Roller_108, origin xyz=-10.239375 0 0.15 rpy=1.5707963 0 0, axis 0 0 1
- added joint Roller_97_109_joint: type continuous, parent base_link, child Roller_109, origin xyz=-10.334625 0 0.15 rpy=1.5707963 0 0, axis 0 0 1
- added joint Roller_97_110_joint: type continuous, parent base_link, child Roller_110, origin xyz=-10.429875000000001 0 0.15 rpy=1.5707963 0 0, axis 0 0 1
- added joint Roller_97_111_joint: type continuous, parent base_link, child Roller_111, origin xyz=-10.525125000000001 0 0.15 rpy=1.5707963 0 0, axis 0 0 1
- added joint Roller_97_112_joint: type continuous, parent base_link, child Roller_112, origin xyz=-10.620375000000001 0 0.15 rpy=1.5707963 0 0, axis 0 0 1
- added joint Roller_97_113_joint: type continuous, parent base_link, child Roller_113, origin xyz=-10.715625 0 0.15 rpy=1.5707963 0 0, axis 0 0 1
- added joint Roller_97_114_joint: type continuous, parent base_link, child Roller_114, origin xyz=-10.810875 0 0.15 rpy=1.5707963 0 0, axis 0 0 1
- added joint Roller_97_115_joint: type continuous, parent base_link, child Roller_115, origin xyz=-10.906125 0 0.15 rpy=1.5707963 0 0, axis 0 0 1
- added joint Roller_97_116_joint: type continuous, parent base_link, child Roller_116, origin xyz=-11.001375 0 0.15 rpy=1.5707963 0 0, axis 0 0 1
- added joint Roller_97_117_joint: type continuous, parent base_link, child Roller_117, origin xyz=-11.096625 0 0.15 rpy=1.5707963 0 0, axis 0 0 1
- added joint Roller_97_118_joint: type continuous, parent base_link, child Roller_118, origin xyz=-11.191875 0 0.15 rpy=1.5707963 0 0, axis 0 0 1
- added joint Roller_97_119_joint: type continuous, parent base_link, child Roller_119, origin xyz=-11.287125 0 0.15 rpy=1.5707963 0 0, axis 0 0 1
- added joint Roller_97_120_joint: type continuous, parent base_link, child Roller_120, origin xyz=-11.382375 0 0.15 rpy=1.5707963 0 0, axis 0 0 1
- added joint Roller_97_121_joint: type continuous, parent base_link, child Roller_121, origin xyz=-11.477625 0 0.15 rpy=1.5707963 0 0, axis 0 0 1
- added joint Roller_97_122_joint: type continuous, parent base_link, child Roller_122, origin xyz=-11.572875 0 0.15 rpy=1.5707963 0 0, axis 0 0 1
- added joint Roller_97_123_joint: type continuous, parent base_link, child Roller_123, origin xyz=-11.668125 0 0.15 rpy=1.5707963 0 0, axis 0 0 1
- added joint Roller_97_124_joint: type continuous, parent base_link, child Roller_124, origin xyz=-11.763375 0 0.15 rpy=1.5707963 0 0, axis 0 0 1
- added joint Roller_97_125_joint: type continuous, parent base_link, child Roller_125, origin xyz=-11.858625 0 0.15 rpy=1.5707963 0 0, axis 0 0 1
- added joint Roller_97_126_joint: type continuous, parent base_link, child Roller_126, origin xyz=-11.953875 0 0.15 rpy=1.5707963 0 0, axis 0 0 1
- added joint Roller_97_127_joint: type continuous, parent base_link, child Roller_127, origin xyz=-12.049125 0 0.15 rpy=1.5707963 0 0, axis 0 0 1
- added joint Roller_97_128_joint: type continuous, parent base_link, child Roller_128, origin xyz=-12.144375 0 0.15 rpy=1.5707963 0 0, axis 0 0 1
- added joint Roller_97_97_joint: type continuous, parent base_link, child Roller_97, origin xyz=-9.191625 0 0.15 rpy=1.570796 0 0, axis 0 0 1
- added joint Roller_97_98_joint: type continuous, parent base_link, child Roller_98, origin xyz=-9.286875 0 0.15 rpy=1.5707963 0 0, axis 0 0 1
- added joint Roller_97_99_joint: type continuous, parent base_link, child Roller_99, origin xyz=-9.382125 0 0.15 rpy=1.5707963 0 0, axis 0 0 1

Commit message: sdf

File: custom40ftStraight.urdf (robot description, URDF)
Before this commit: robot roller_conveyor_40ft, 131 links, 130 joints
Links:
- added link base_footprint
Joints:
- added joint base_link: type fixed, parent base_footprint, child base_link, origin xyz=0 0 0 rpy=0 0 0
