Commit message: clean up

File: custom40ftStraight.xacro (robot description, xacro)
@@ -91,15 +91,4 @@
         <axis xyz="0 0 1"/>
     </joint>
-    <!-- Rollers -->
-    <!-- 56 Rollers, Spacing = 12.192m / 56 spaces ≈ 0.2177m apart -->
-    <!-- Define 14 Rollers -->
-    <!-- Roller Diameter = 50.8mm (0.0508m), Length = 4ft (1.219m) -->
-    <!-- Rollers List -->
-    <!-- Each roller has a continuous joint allowing unlimited rotation -->
-    <!-- Looping manually without macros -->
-    <!-- 14 Rollers Definition -->
-    <!-- Index i ∈ [0, 13], Position Y = -0.762 + i * 0.117m -->
-    <!-- Roller Definition Loop -->
-    <!-- Define 14 rollers manually -->
     <!-- Start Roller Definitions -->
     <!-- In between rollers, starting from #1->#32 -->
@@ -145,5 +134,5 @@
             <collision>
                 <geometry>
-                    <cylinder radius="0.05" length="1.219"/>
+                    <cylinder radius="0.025" length="1.219"/>
                 </geometry>
             </collision>
@@ -204,5 +193,5 @@
             <collision>
                 <geometry>
-                    <cylinder radius="0.05" length="1.219"/>
+                    <cylinder radius="0.025" length="1.219"/>
                 </geometry>
             </collision>
@@ -263,5 +252,5 @@
             <collision>
                 <geometry>
-                    <cylinder radius="0.05" length="1.219"/>
+                    <cylinder radius="0.025" length="1.219"/>
                 </geometry>
             </collision>
@@ -322,5 +311,5 @@
             <collision>
                 <geometry>
-                    <cylinder radius="0.05" length="1.219"/>
+                    <cylinder radius="0.025" length="1.219"/>
                 </geometry>
             </collision>

Commit message: remove name

File: custom40ftStraight.xacro (robot description, xacro)
@@ -122,5 +122,5 @@
     </joint>
     <!-- Roller #2->#32 -->
-    <xacro:macro name="roller1st5ft" params="name rollerNum">
+    <xacro:macro name="roller1st5ft" params="rollerNum">
         <link name="Roller_${rollerNum}">
             <visual>
@@ -181,5 +181,5 @@
     </joint>
     <!-- Roller #34->#64 -->
-    <xacro:macro name="roller2nd5ft" params="name rollerNum">
+    <xacro:macro name="roller2nd5ft" params="rollerNum">
         <link name="Roller_${rollerNum}">
             <visual>
@@ -240,5 +240,5 @@
     </joint>
     <!-- Roller #66->#96 -->
-    <xacro:macro name="roller3rd5ft" params="name rollerNum">
+    <xacro:macro name="roller3rd5ft" params="rollerNum">
         <link name="Roller_${rollerNum}">
             <visual>
@@ -299,5 +299,5 @@
     </joint>
     <!-- Roller #98->#128 -->
-    <xacro:macro name="roller4th5ft" params="name rollerNum">
+    <xacro:macro name="roller4th5ft" params="rollerNum">
         <link name="Roller_${rollerNum}">
             <visual>

Commit message: change xacro

File: custom40ftStraight.xacro (robot description, xacro)
@@ -113,5 +113,5 @@
         </inertial>
     </link>
-    <joint name="Roller_1_joint" type="continuous">
+    <joint name="Roller_1_1_joint" type="continuous">
         <parent link="base_link"/>
         <child link="Roller_1"/>
@@ -141,5 +141,5 @@
             </inertial>
         </link>
-        <joint name="Roller_${rollerNum}_joint" type="continuous">
+        <joint name="Roller_1_${rollerNum}_joint" type="continuous">
             <parent link="base_link"/>
             <child link="Roller_${rollerNum}"/>
@@ -171,5 +171,5 @@
         </inertial>
     </link>
-    <joint name="Roller_33_joint" type="continuous">
+    <joint name="Roller_33_33_joint" type="continuous">
         <parent link="base_link"/>
         <child link="Roller_33"/>
@@ -199,5 +199,5 @@
             </inertial>
         </link>
-        <joint name="Roller_${rollerNum}_joint" type="continuous">
+        <joint name="Roller_33_${rollerNum}_joint" type="continuous">
             <parent link="base_link"/>
             <child link="Roller_${rollerNum}"/>
@@ -229,5 +229,5 @@
         </inertial>
     </link>
-    <joint name="Roller_65_joint" type="continuous">
+    <joint name="Roller_65_65_joint" type="continuous">
         <parent link="base_link"/>
         <child link="Roller_65"/>
@@ -257,5 +257,5 @@
             </inertial>
         </link>
-        <joint name="Roller_${rollerNum}_joint" type="continuous">
+        <joint name="Roller_65_${rollerNum}_joint" type="continuous">
             <parent link="base_link"/>
             <child link="Roller_${rollerNum}"/>
@@ -287,5 +287,5 @@
         </inertial>
     </link>
-    <joint name="Roller_97_joint" type="continuous">
+    <joint name="Roller_97_97_joint" type="continuous">
         <parent link="base_link"/>
         <child link="Roller_97"/>
@@ -315,5 +315,5 @@
             </inertial>
         </link>
-        <joint name="Roller_${rollerNum}_joint" type="continuous">
+        <joint name="Roller_97_${rollerNum}_joint" type="continuous">
             <parent link="base_link"/>
             <child link="Roller_${rollerNum}"/>

Commit message: Update custom40ftStraight.xacro

File: custom40ftStraight.xacro (robot description, xacro)
@@ -118,5 +118,5 @@
         <origin xyz="-${roller_pitch/2} 0 0.15" rpy="1.570796 0 0"/>
         <axis xyz="0 0 1"/>
-        <dynamics damping="0.1" friction="0.2"/>
+        <dynamics damping="1.0" friction="0.0"/>
     </joint>
     <!-- Roller #2->#32 -->
@@ -146,6 +146,5 @@
             <origin xyz="-${(rollerNum-1)*roller_pitch + roller_pitch/2} 0 0.15" rpy="${pi/2} 0 0"/>
             <axis xyz="0 0 1"/>
-            <dynamics damping="0.1" friction="0.2"/>
-            <mimic joint="Roller_1_joint" multiplier="1" offset="0" />
+            <dynamics damping="1.0" friction="0.0"/>
         </joint>
     </xacro:macro>
@@ -176,5 +175,5 @@
         <origin xyz="-${(32)*roller_pitch + roller_pitch/2} 0 0.15" rpy="1.570796 0 0"/>
         <axis xyz="0 0 1"/>
-        <dynamics damping="0.1" friction="0.2"/>
+        <dynamics damping="1.0" friction="0.0"/>
     </joint>
     <!-- Roller #34->#64 -->
@@ -204,6 +203,5 @@
             <origin xyz="-${(rollerNum-1)*roller_pitch + roller_pitch/2} 0 0.15" rpy="${pi/2} 0 0"/>
             <axis xyz="0 0 1"/>
-            <dynamics damping="0.1" friction="0.2"/>
-            <mimic joint="Roller_33_joint" multiplier="1" offset="0" />
+            <dynamics damping="1.0" friction="0.0"/>
         </joint>
     </xacro:macro>
@@ -234,5 +232,5 @@
         <origin xyz="-${(64)*roller_pitch + roller_pitch/2} 0 0.15" rpy="1.570796 0 0"/>
         <axis xyz="0 0 1"/>
-        <dynamics damping="0.1" friction="0.2"/>
+        <dynamics damping="1.0" friction="0.0"/>
     </joint>
     <!-- Roller #66->#96 -->
@@ -262,6 +260,5 @@
             <origin xyz="-${(rollerNum-1)*roller_pitch + roller_pitch/2} 0 0.15" rpy="${pi/2} 0 0"/>
             <axis xyz="0 0 1"/>
-            <dynamics damping="0.1" friction="0.2"/>
-            <mimic joint="Roller_65_joint" multiplier="1" offset="0" />
+            <dynamics damping="1.0" friction="0.0"/>
         </joint>
     </xacro:macro>
@@ -292,5 +289,5 @@
         <origin xyz="-${(96)*roller_pitch + roller_pitch/2} 0 0.15" rpy="1.570796 0 0"/>
         <axis xyz="0 0 1"/>
-        <dynamics damping="0.1" friction="0.2"/>
+        <dynamics damping="1.0" friction="0.0"/>
     </joint>
     <!-- Roller #98->#128 -->
@@ -320,6 +317,5 @@
             <origin xyz="-${(rollerNum-1)*roller_pitch + roller_pitch/2} 0 0.15" rpy="${pi/2} 0 0"/>
             <axis xyz="0 0 1"/>
-            <dynamics damping="0.1" friction="0.2"/>
-            <mimic joint="Roller_97_joint" multiplier="1" offset="0" />
+            <dynamics damping="1.0" friction="0.0"/>
         </joint>
     </xacro:macro>

Commit message: xacro v2

File: custom40ftStraight.xacro (robot description, xacro)
@@ -10,4 +10,10 @@
     <xacro:property name="pi" value="3.1415926"/>
     <xacro:property name="roller_spacing" value="${conveyor_length / (roller_count)}"/>
+    <link name="base_footprint"/>
+    <joint name="base_link" type="fixed">
+        <origin rpy="0 0 0" xyz="0 0 0"/>
+        <parent link="base_footprint"/>
+        <child link="base_link"/>
+    </joint>
     <!-- Base Frame -->
     <link name="base_link">
