Commit message: add tall v3

File: custom40ftStraight_v3.urdf (robot description, URDF)
Before this commit: robot roller_conveyor_40ft, 132 links, 131 joints
Links:
- link base_link: geometry collision box size=12.192 1.219 2.0; visual box size=12.192 1.219 2.0
- link leftFrame: geometry collision box size=12.192 0.05 2.5; visual box size=12.192 0.05 2.5
- link rightFrame: geometry collision box size=12.192 0.05 2.5; visual box size=12.192 0.05 2.5
Joints:
- joint Roller_113_113_joint: origin xyz=-10.715625 0 0.15 rpy=1.570796 0 0 -> xyz=-10.715625 0 1.15 rpy=1.570796 0 0
- joint Roller_113_114_joint: mimic joint=Roller_113_113_joint multiplier=1 offset=0 -> (none); origin xyz=-10.810875 0 0.15 rpy=1.5707963 0 0 -> xyz=-10.810875 0 1.15 rpy=1.5707963 0 0
- joint Roller_113_115_joint: mimic joint=Roller_113_113_joint multiplier=1 offset=0 -> (none); origin xyz=-10.906125 0 0.15 rpy=1.5707963 0 0 -> xyz=-10.906125 0 1.15 rpy=1.5707963 0 0
- joint Roller_113_116_joint: mimic joint=Roller_113_113_joint multiplier=1 offset=0 -> (none); origin xyz=-11.001375 0 0.15 rpy=1.5707963 0 0 -> xyz=-11.001375 0 1.15 rpy=1.5707963 0 0
- joint Roller_113_117_joint: mimic joint=Roller_113_113_joint multiplier=1 offset=0 -> (none); origin xyz=-11.096625 0 0.15 rpy=1.5707963 0 0 -> xyz=-11.096625 0 1.15 rpy=1.5707963 0 0
- joint Roller_113_118_joint: mimic joint=Roller_113_113_joint multiplier=1 offset=0 -> (none); origin xyz=-11.191875 0 0.15 rpy=1.5707963 0 0 -> xyz=-11.191875 0 1.15 rpy=1.5707963 0 0
- joint Roller_113_119_joint: mimic joint=Roller_113_113_joint multiplier=1 offset=0 -> (none); origin xyz=-11.287125 0 0.15 rpy=1.5707963 0 0 -> xyz=-11.287125 0 1.15 rpy=1.5707963 0 0
- joint Roller_113_120_joint: mimic joint=Roller_113_113_joint multiplier=1 offset=0 -> (none); origin xyz=-11.382375 0 0.15 rpy=1.5707963 0 0 -> xyz=-11.382375 0 1.15 rpy=1.5707963 0 0
- joint Roller_113_121_joint: mimic joint=Roller_113_113_joint multiplier=1 offset=0 -> (none); origin xyz=-11.477625 0 0.15 rpy=1.5707963 0 0 -> xyz=-11.477625 0 1.15 rpy=1.5707963 0 0
- joint Roller_113_122_joint: mimic joint=Roller_113_113_joint multiplier=1 offset=0 -> (none); origin xyz=-11.572875 0 0.15 rpy=1.5707963 0 0 -> xyz=-11.572875 0 1.15 rpy=1.5707963 0 0
- joint Roller_113_123_joint: mimic joint=Roller_113_113_joint multiplier=1 offset=0 -> (none); origin xyz=-11.668125 0 0.15 rpy=1.5707963 0 0 -> xyz=-11.668125 0 1.15 rpy=1.5707963 0 0
- joint Roller_113_124_joint: mimic joint=Roller_113_113_joint multiplier=1 offset=0 -> (none); origin xyz=-11.763375 0 0.15 rpy=1.5707963 0 0 -> xyz=-11.763375 0 1.15 rpy=1.5707963 0 0
- joint Roller_113_125_joint: mimic joint=Roller_113_113_joint multiplier=1 offset=0 -> (none); origin xyz=-11.858625 0 0.15 rpy=1.5707963 0 0 -> xyz=-11.858625 0 1.15 rpy=1.5707963 0 0
- joint Roller_113_126_joint: mimic joint=Roller_113_113_joint multiplier=1 offset=0 -> (none); origin xyz=-11.953875 0 0.15 rpy=1.5707963 0 0 -> xyz=-11.953875 0 1.15 rpy=1.5707963 0 0
- joint Roller_113_127_joint: mimic joint=Roller_113_113_joint multiplier=1 offset=0 -> (none); origin xyz=-12.049125 0 0.15 rpy=1.5707963 0 0 -> xyz=-12.049125 0 1.15 rpy=1.5707963 0 0
- joint Roller_113_128_joint: mimic joint=Roller_113_113_joint multiplier=1 offset=0 -> (none); origin xyz=-12.144375 0 0.15 rpy=1.5707963 0 0 -> xyz=-12.144375 0 1.15 rpy=1.5707963 0 0
- joint Roller_17_17_joint: origin xyz=-1.571625 0 0.15 rpy=1.570796 0 0 -> xyz=-1.571625 0 1.15 rpy=1.570796 0 0
- joint Roller_17_18_joint: mimic joint=Roller_17_17_joint multiplier=1 offset=0 -> (none); origin xyz=-1.666875 0 0.15 rpy=1.5707963 0 0 -> xyz=-1.666875 0 1.15 rpy=1.5707963 0 0
- joint Roller_17_19_joint: mimic joint=Roller_17_17_joint multiplier=1 offset=0 -> (none); origin xyz=-1.7621250000000002 0 0.15 rpy=1.5707963 0 0 -> xyz=-1.7621250000000002 0 1.15 rpy=1.5707963 0 0
- joint Roller_17_20_joint: mimic joint=Roller_17_17_joint multiplier=1 offset=0 -> (none); origin xyz=-1.857375 0 0.15 rpy=1.5707963 0 0 -> xyz=-1.857375 0 1.15 rpy=1.5707963 0 0
- joint Roller_17_21_joint: mimic joint=Roller_17_17_joint multiplier=1 offset=0 -> (none); origin xyz=-1.952625 0 0.15 rpy=1.5707963 0 0 -> xyz=-1.952625 0 1.15 rpy=1.5707963 0 0
- joint Roller_17_22_joint: mimic joint=Roller_17_17_joint multiplier=1 offset=0 -> (none); origin xyz=-2.047875 0 0.15 rpy=1.5707963 0 0 -> xyz=-2.047875 0 1.15 rpy=1.5707963 0 0
- joint Roller_17_23_joint: mimic joint=Roller_17_17_joint multiplier=1 offset=0 -> (none); origin xyz=-2.143125 0 0.15 rpy=1.5707963 0 0 -> xyz=-2.143125 0 1.15 rpy=1.5707963 0 0
- joint Roller_17_24_joint: mimic joint=Roller_17_17_joint multiplier=1 offset=0 -> (none); origin xyz=-2.238375 0 0.15 rpy=1.5707963 0 0 -> xyz=-2.238375 0 1.15 rpy=1.5707963 0 0
- joint Roller_17_25_joint: mimic joint=Roller_17_17_joint multiplier=1 offset=0 -> (none); origin xyz=-2.333625 0 0.15 rpy=1.5707963 0 0 -> xyz=-2.333625 0 1.15 rpy=1.5707963 0 0
- joint Roller_17_26_joint: mimic joint=Roller_17_17_joint multiplier=1 offset=0 -> (none); origin xyz=-2.428875 0 0.15 rpy=1.5707963 0 0 -> xyz=-2.428875 0 1.15 rpy=1.5707963 0 0
- joint Roller_17_27_joint: mimic joint=Roller_17_17_joint multiplier=1 offset=0 -> (none); origin xyz=-2.524125 0 0.15 rpy=1.5707963 0 0 -> xyz=-2.524125 0 1.15 rpy=1.5707963 0 0
- joint Roller_17_28_joint: mimic joint=Roller_17_17_joint multiplier=1 offset=0 -> (none); origin xyz=-2.6193750000000002 0 0.15 rpy=1.5707963 0 0 -> xyz=-2.6193750000000002 0 1.15 rpy=1.5707963 0 0
- joint Roller_17_29_joint: mimic joint=Roller_17_17_joint multiplier=1 offset=0 -> (none); origin xyz=-2.714625 0 0.15 rpy=1.5707963 0 0 -> xyz=-2.714625 0 1.15 rpy=1.5707963 0 0
- joint Roller_17_30_joint: mimic joint=Roller_17_17_joint multiplier=1 offset=0 -> (none); origin xyz=-2.809875 0 0.15 rpy=1.5707963 0 0 -> xyz=-2.809875 0 1.15 rpy=1.5707963 0 0
- joint Roller_17_31_joint: mimic joint=Roller_17_17_joint multiplier=1 offset=0 -> (none); origin xyz=-2.905125 0 0.15 rpy=1.5707963 0 0 -> xyz=-2.905125 0 1.15 rpy=1.5707963 0 0
- joint Roller_17_32_joint: mimic joint=Roller_17_17_joint multiplier=1 offset=0 -> (none); origin xyz=-3.000375 0 0.15 rpy=1.5707963 0 0 -> xyz=-3.000375 0 1.15 rpy=1.5707963 0 0
- joint Roller_1_10_joint: mimic joint=Roller_1_1_joint multiplier=1 offset=0 -> (none); origin xyz=-0.9048750000000001 0 0.15 rpy=1.5707963 0 0 -> xyz=-0.9048750000000001 0 1.15 rpy=1.5707963 0 0
- joint Roller_1_11_joint: mimic joint=Roller_1_1_joint multiplier=1 offset=0 -> (none); origin xyz=-1.000125 0 0.15 rpy=1.5707963 0 0 -> xyz=-1.000125 0 1.15 rpy=1.5707963 0 0
- joint Roller_1_12_joint: mimic joint=Roller_1_1_joint multiplier=1 offset=0 -> (none); origin xyz=-1.095375 0 0.15 rpy=1.5707963 0 0 -> xyz=-1.095375 0 1.15 rpy=1.5707963 0 0
- joint Roller_1_13_joint: mimic joint=Roller_1_1_joint multiplier=1 offset=0 -> (none); origin xyz=-1.190625 0 0.15 rpy=1.5707963 0 0 -> xyz=-1.190625 0 1.15 rpy=1.5707963 0 0
- joint Roller_1_14_joint: mimic joint=Roller_1_1_joint multiplier=1 offset=0 -> (none); origin xyz=-1.285875 0 0.15 rpy=1.5707963 0 0 -> xyz=-1.285875 0 1.15 rpy=1.5707963 0 0
- joint Roller_1_15_joint: mimic joint=Roller_1_1_joint multiplier=1 offset=0 -> (none); origin xyz=-1.381125 0 0.15 rpy=1.5707963 0 0 -> xyz=-1.381125 0 1.15 rpy=1.5707963 0 0
- joint Roller_1_16_joint: mimic joint=Roller_1_1_joint multiplier=1 offset=0 -> (none); origin xyz=-1.476375 0 0.15 rpy=1.5707963 0 0 -> xyz=-1.476375 0 1.15 rpy=1.5707963 0 0
- joint Roller_1_1_joint: origin xyz=-0.047625 0 0.15 rpy=1.570796 0 0 -> xyz=-0.047625 0 1.15 rpy=1.570796 0 0
- joint Roller_1_2_joint: mimic joint=Roller_1_1_joint multiplier=1 offset=0 -> (none); origin xyz=-0.142875 0 0.15 rpy=1.5707963 0 0 -> xyz=-0.142875 0 1.15 rpy=1.5707963 0 0
- joint Roller_1_3_joint: mimic joint=Roller_1_1_joint multiplier=1 offset=0 -> (none); origin xyz=-0.238125 0 0.15 rpy=1.5707963 0 0 -> xyz=-0.238125 0 1.15 rpy=1.5707963 0 0
- joint Roller_1_4_joint: mimic joint=Roller_1_1_joint multiplier=1 offset=0 -> (none); origin xyz=-0.333375 0 0.15 rpy=1.5707963 0 0 -> xyz=-0.333375 0 1.15 rpy=1.5707963 0 0
- joint Roller_1_5_joint: mimic joint=Roller_1_1_joint multiplier=1 offset=0 -> (none); origin xyz=-0.42862500000000003 0 0.15 rpy=1.5707963 0 0 -> xyz=-0.42862500000000003 0 1.15 rpy=1.5707963 0 0
- joint Roller_1_6_joint: mimic joint=Roller_1_1_joint multiplier=1 offset=0 -> (none); origin xyz=-0.523875 0 0.15 rpy=1.5707963 0 0 -> xyz=-0.523875 0 1.15 rpy=1.5707963 0 0
- joint Roller_1_7_joint: mimic joint=Roller_1_1_joint multiplier=1 offset=0 -> (none); origin xyz=-0.619125 0 0.15 rpy=1.5707963 0 0 -> xyz=-0.619125 0 1.15 rpy=1.5707963 0 0
- joint Roller_1_8_joint: mimic joint=Roller_1_1_joint multiplier=1 offset=0 -> (none); origin xyz=-0.714375 0 0.15 rpy=1.5707963 0 0 -> xyz=-0.714375 0 1.15 rpy=1.5707963 0 0
- joint Roller_1_9_joint: mimic joint=Roller_1_1_joint multiplier=1 offset=0 -> (none); origin xyz=-0.809625 0 0.15 rpy=1.5707963 0 0 -> xyz=-0.809625 0 1.15 rpy=1.5707963 0 0
- joint Roller_33_33_joint: origin xyz=-3.095625 0 0.15 rpy=1.570796 0 0 -> xyz=-3.095625 0 1.15 rpy=1.570796 0 0
- joint Roller_33_34_joint: mimic joint=Roller_33_33_joint multiplier=1 offset=0 -> (none); origin xyz=-3.190875 0 0.15 rpy=1.5707963 0 0 -> xyz=-3.190875 0 1.15 rpy=1.5707963 0 0
- joint Roller_33_35_joint: mimic joint=Roller_33_33_joint multiplier=1 offset=0 -> (none); origin xyz=-3.286125 0 0.15 rpy=1.5707963 0 0 -> xyz=-3.286125 0 1.15 rpy=1.5707963 0 0
- joint Roller_33_36_joint: mimic joint=Roller_33_33_joint multiplier=1 offset=0 -> (none); origin xyz=-3.3813750000000002 0 0.15 rpy=1.5707963 0 0 -> xyz=-3.3813750000000002 0 1.15 rpy=1.5707963 0 0
- joint Roller_33_37_joint: mimic joint=Roller_33_33_joint multiplier=1 offset=0 -> (none); origin xyz=-3.4766250000000003 0 0.15 rpy=1.5707963 0 0 -> xyz=-3.4766250000000003 0 1.15 rpy=1.5707963 0 0
- joint Roller_33_38_joint: mimic joint=Roller_33_33_joint multiplier=1 offset=0 -> (none); origin xyz=-3.571875 0 0.15 rpy=1.5707963 0 0 -> xyz=-3.571875 0 1.15 rpy=1.5707963 0 0
- joint Roller_33_39_joint: mimic joint=Roller_33_33_joint multiplier=1 offset=0 -> (none); origin xyz=-3.667125 0 0.15 rpy=1.5707963 0 0 -> xyz=-3.667125 0 1.15 rpy=1.5707963 0 0
- joint Roller_33_40_joint: mimic joint=Roller_33_33_joint multiplier=1 offset=0 -> (none); origin xyz=-3.762375 0 0.15 rpy=1.5707963 0 0 -> xyz=-3.762375 0 1.15 rpy=1.5707963 0 0
- joint Roller_33_41_joint: mimic joint=Roller_33_33_joint multiplier=1 offset=0 -> (none); origin xyz=-3.857625 0 0.15 rpy=1.5707963 0 0 -> xyz=-3.857625 0 1.15 rpy=1.5707963 0 0
- joint Roller_33_42_joint: mimic joint=Roller_33_33_joint multiplier=1 offset=0 -> (none); origin xyz=-3.952875 0 0.15 rpy=1.5707963 0 0 -> xyz=-3.952875 0 1.15 rpy=1.5707963 0 0
- joint Roller_33_43_joint: mimic joint=Roller_33_33_joint multiplier=1 offset=0 -> (none); origin xyz=-4.048125 0 0.15 rpy=1.5707963 0 0 -> xyz=-4.048125 0 1.15 rpy=1.5707963 0 0
- joint Roller_33_44_joint: mimic joint=Roller_33_33_joint multiplier=1 offset=0 -> (none); origin xyz=-4.143375 0 0.15 rpy=1.5707963 0 0 -> xyz=-4.143375 0 1.15 rpy=1.5707963 0 0
- joint Roller_33_45_joint: mimic joint=Roller_33_33_joint multiplier=1 offset=0 -> (none); origin xyz=-4.238625 0 0.15 rpy=1.5707963 0 0 -> xyz=-4.238625 0 1.15 rpy=1.5707963 0 0
- joint Roller_33_46_joint: mimic joint=Roller_33_33_joint multiplier=1 offset=0 -> (none); origin xyz=-4.333875 0 0.15 rpy=1.5707963 0 0 -> xyz=-4.333875 0 1.15 rpy=1.5707963 0 0
- joint Roller_33_47_joint: mimic joint=Roller_33_33_joint multiplier=1 offset=0 -> (none); origin xyz=-4.429125 0 0.15 rpy=1.5707963 0 0 -> xyz=-4.429125 0 1.15 rpy=1.5707963 0 0
- joint Roller_33_48_joint: mimic joint=Roller_33_33_joint multiplier=1 offset=0 -> (none); origin xyz=-4.524375 0 0.15 rpy=1.5707963 0 0 -> xyz=-4.524375 0 1.15 rpy=1.5707963 0 0
- joint Roller_49_49_joint: origin xyz=-4.619625 0 0.15 rpy=1.570796 0 0 -> xyz=-4.619625 0 1.15 rpy=1.570796 0 0
- joint Roller_49_50_joint: mimic joint=Roller_49_49_joint multiplier=1 offset=0 -> (none); origin xyz=-4.714875 0 0.15 rpy=1.5707963 0 0 -> xyz=-4.714875 0 1.15 rpy=1.5707963 0 0
- joint Roller_49_51_joint: mimic joint=Roller_49_49_joint multiplier=1 offset=0 -> (none); origin xyz=-4.810125 0 0.15 rpy=1.5707963 0 0 -> xyz=-4.810125 0 1.15 rpy=1.5707963 0 0
- joint Roller_49_52_joint: mimic joint=Roller_49_49_joint multiplier=1 offset=0 -> (none); origin xyz=-4.905375 0 0.15 rpy=1.5707963 0 0 -> xyz=-4.905375 0 1.15 rpy=1.5707963 0 0
- joint Roller_49_53_joint: mimic joint=Roller_49_49_joint multiplier=1 offset=0 -> (none); origin xyz=-5.000625 0 0.15 rpy=1.5707963 0 0 -> xyz=-5.000625 0 1.15 rpy=1.5707963 0 0
- joint Roller_49_54_joint: mimic joint=Roller_49_49_joint multiplier=1 offset=0 -> (none); origin xyz=-5.095875 0 0.15 rpy=1.5707963 0 0 -> xyz=-5.095875 0 1.15 rpy=1.5707963 0 0
- joint Roller_49_55_joint: mimic joint=Roller_49_49_joint multiplier=1 offset=0 -> (none); origin xyz=-5.191125 0 0.15 rpy=1.5707963 0 0 -> xyz=-5.191125 0 1.15 rpy=1.5707963 0 0
- joint Roller_49_56_joint: mimic joint=Roller_49_49_joint multiplier=1 offset=0 -> (none); origin xyz=-5.2863750000000005 0 0.15 rpy=1.5707963 0 0 -> xyz=-5.2863750000000005 0 1.15 rpy=1.5707963 0 0
- joint Roller_49_57_joint: mimic joint=Roller_49_49_joint multiplier=1 offset=0 -> (none); origin xyz=-5.381625 0 0.15 rpy=1.5707963 0 0 -> xyz=-5.381625 0 1.15 rpy=1.5707963 0 0
- joint Roller_49_58_joint: mimic joint=Roller_49_49_joint multiplier=1 offset=0 -> (none); origin xyz=-5.476875 0 0.15 rpy=1.5707963 0 0 -> xyz=-5.476875 0 1.15 rpy=1.5707963 0 0
- joint Roller_49_59_joint: mimic joint=Roller_49_49_joint multiplier=1 offset=0 -> (none); origin xyz=-5.572125 0 0.15 rpy=1.5707963 0 0 -> xyz=-5.572125 0 1.15 rpy=1.5707963 0 0
- joint Roller_49_60_joint: mimic joint=Roller_49_49_joint multiplier=1 offset=0 -> (none); origin xyz=-5.667375 0 0.15 rpy=1.5707963 0 0 -> xyz=-5.667375 0 1.15 rpy=1.5707963 0 0
- joint Roller_49_61_joint: mimic joint=Roller_49_49_joint multiplier=1 offset=0 -> (none); origin xyz=-5.762625 0 0.15 rpy=1.5707963 0 0 -> xyz=-5.762625 0 1.15 rpy=1.5707963 0 0
- joint Roller_49_62_joint: mimic joint=Roller_49_49_joint multiplier=1 offset=0 -> (none); origin xyz=-5.857875 0 0.15 rpy=1.5707963 0 0 -> xyz=-5.857875 0 1.15 rpy=1.5707963 0 0
- joint Roller_49_63_joint: mimic joint=Roller_49_49_joint multiplier=1 offset=0 -> (none); origin xyz=-5.953125 0 0.15 rpy=1.5707963 0 0 -> xyz=-5.953125 0 1.15 rpy=1.5707963 0 0
- joint Roller_49_64_joint: mimic joint=Roller_49_49_joint multiplier=1 offset=0 -> (none); origin xyz=-6.048375 0 0.15 rpy=1.5707963 0 0 -> xyz=-6.048375 0 1.15 rpy=1.5707963 0 0
- joint Roller_65_65_joint: origin xyz=-6.143625 0 0.15 rpy=1.570796 0 0 -> xyz=-6.143625 0 1.15 rpy=1.570796 0 0
- joint Roller_65_66_joint: mimic joint=Roller_65_65_joint multiplier=1 offset=0 -> (none); origin xyz=-6.238875 0 0.15 rpy=1.5707963 0 0 -> xyz=-6.238875 0 1.15 rpy=1.5707963 0 0
- joint Roller_65_67_joint: mimic joint=Roller_65_65_joint multiplier=1 offset=0 -> (none); origin xyz=-6.334125 0 0.15 rpy=1.5707963 0 0 -> xyz=-6.334125 0 1.15 rpy=1.5707963 0 0
- joint Roller_65_68_joint: mimic joint=Roller_65_65_joint multiplier=1 offset=0 -> (none); origin xyz=-6.429375 0 0.15 rpy=1.5707963 0 0 -> xyz=-6.429375 0 1.15 rpy=1.5707963 0 0
- joint Roller_65_69_joint: mimic joint=Roller_65_65_joint multiplier=1 offset=0 -> (none); origin xyz=-6.524625 0 0.15 rpy=1.5707963 0 0 -> xyz=-6.524625 0 1.15 rpy=1.5707963 0 0
- joint Roller_65_70_joint: mimic joint=Roller_65_65_joint multiplier=1 offset=0 -> (none); origin xyz=-6.619875 0 0.15 rpy=1.5707963 0 0 -> xyz=-6.619875 0 1.15 rpy=1.5707963 0 0
- joint Roller_65_71_joint: mimic joint=Roller_65_65_joint multiplier=1 offset=0 -> (none); origin xyz=-6.7151250000000005 0 0.15 rpy=1.5707963 0 0 -> xyz=-6.7151250000000005 0 1.15 rpy=1.5707963 0 0
- joint Roller_65_72_joint: mimic joint=Roller_65_65_joint multiplier=1 offset=0 -> (none); origin xyz=-6.8103750000000005 0 0.15 rpy=1.5707963 0 0 -> xyz=-6.8103750000000005 0 1.15 rpy=1.5707963 0 0
- joint Roller_65_73_joint: mimic joint=Roller_65_65_joint multiplier=1 offset=0 -> (none); origin xyz=-6.905625000000001 0 0.15 rpy=1.5707963 0 0 -> xyz=-6.905625000000001 0 1.15 rpy=1.5707963 0 0
- joint Roller_65_74_joint: mimic joint=Roller_65_65_joint multiplier=1 offset=0 -> (none); origin xyz=-7.000875 0 0.15 rpy=1.5707963 0 0 -> xyz=-7.000875 0 1.15 rpy=1.5707963 0 0
- joint Roller_65_75_joint: mimic joint=Roller_65_65_joint multiplier=1 offset=0 -> (none); origin xyz=-7.096125 0 0.15 rpy=1.5707963 0 0 -> xyz=-7.096125 0 1.15 rpy=1.5707963 0 0
- joint Roller_65_76_joint: mimic joint=Roller_65_65_joint multiplier=1 offset=0 -> (none); origin xyz=-7.191375 0 0.15 rpy=1.5707963 0 0 -> xyz=-7.191375 0 1.15 rpy=1.5707963 0 0
- joint Roller_65_77_joint: mimic joint=Roller_65_65_joint multiplier=1 offset=0 -> (none); origin xyz=-7.286625 0 0.15 rpy=1.5707963 0 0 -> xyz=-7.286625 0 1.15 rpy=1.5707963 0 0
- joint Roller_65_78_joint: mimic joint=Roller_65_65_joint multiplier=1 offset=0 -> (none); origin xyz=-7.381875 0 0.15 rpy=1.5707963 0 0 -> xyz=-7.381875 0 1.15 rpy=1.5707963 0 0
- joint Roller_65_79_joint: mimic joint=Roller_65_65_joint multiplier=1 offset=0 -> (none); origin xyz=-7.477125 0 0.15 rpy=1.5707963 0 0 -> xyz=-7.477125 0 1.15 rpy=1.5707963 0 0
- joint Roller_65_80_joint: mimic joint=Roller_65_65_joint multiplier=1 offset=0 -> (none); origin xyz=-7.572375 0 0.15 rpy=1.5707963 0 0 -> xyz=-7.572375 0 1.15 rpy=1.5707963 0 0
- joint Roller_81_81_joint: origin xyz=-7.667625 0 0.15 rpy=1.570796 0 0 -> xyz=-7.667625 0 1.15 rpy=1.570796 0 0
- joint Roller_81_82_joint: mimic joint=Roller_81_81_joint multiplier=1 offset=0 -> (none); origin xyz=-7.762875 0 0.15 rpy=1.5707963 0 0 -> xyz=-7.762875 0 1.15 rpy=1.5707963 0 0
- joint Roller_81_83_joint: mimic joint=Roller_81_81_joint multiplier=1 offset=0 -> (none); origin xyz=-7.858125 0 0.15 rpy=1.5707963 0 0 -> xyz=-7.858125 0 1.15 rpy=1.5707963 0 0
- joint Roller_81_84_joint: mimic joint=Roller_81_81_joint multiplier=1 offset=0 -> (none); origin xyz=-7.953375 0 0.15 rpy=1.5707963 0 0 -> xyz=-7.953375 0 1.15 rpy=1.5707963 0 0
- joint Roller_81_85_joint: mimic joint=Roller_81_81_joint multiplier=1 offset=0 -> (none); origin xyz=-8.048625 0 0.15 rpy=1.5707963 0 0 -> xyz=-8.048625 0 1.15 rpy=1.5707963 0 0
- joint Roller_81_86_joint: mimic joint=Roller_81_81_joint multiplier=1 offset=0 -> (none); origin xyz=-8.143875 0 0.15 rpy=1.5707963 0 0 -> xyz=-8.143875 0 1.15 rpy=1.5707963 0 0
- joint Roller_81_87_joint: mimic joint=Roller_81_81_joint multiplier=1 offset=0 -> (none); origin xyz=-8.239125 0 0.15 rpy=1.5707963 0 0 -> xyz=-8.239125 0 1.15 rpy=1.5707963 0 0
- joint Roller_81_88_joint: mimic joint=Roller_81_81_joint multiplier=1 offset=0 -> (none); origin xyz=-8.334375 0 0.15 rpy=1.5707963 0 0 -> xyz=-8.334375 0 1.15 rpy=1.5707963 0 0
- joint Roller_81_89_joint: mimic joint=Roller_81_81_joint multiplier=1 offset=0 -> (none); origin xyz=-8.429625 0 0.15 rpy=1.5707963 0 0 -> xyz=-8.429625 0 1.15 rpy=1.5707963 0 0
- joint Roller_81_90_joint: mimic joint=Roller_81_81_joint multiplier=1 offset=0 -> (none); origin xyz=-8.524875 0 0.15 rpy=1.5707963 0 0 -> xyz=-8.524875 0 1.15 rpy=1.5707963 0 0
- joint Roller_81_91_joint: mimic joint=Roller_81_81_joint multiplier=1 offset=0 -> (none); origin xyz=-8.620125 0 0.15 rpy=1.5707963 0 0 -> xyz=-8.620125 0 1.15 rpy=1.5707963 0 0
- joint Roller_81_92_joint: mimic joint=Roller_81_81_joint multiplier=1 offset=0 -> (none); origin xyz=-8.715375 0 0.15 rpy=1.5707963 0 0 -> xyz=-8.715375 0 1.15 rpy=1.5707963 0 0
- joint Roller_81_93_joint: mimic joint=Roller_81_81_joint multiplier=1 offset=0 -> (none); origin xyz=-8.810625 0 0.15 rpy=1.5707963 0 0 -> xyz=-8.810625 0 1.15 rpy=1.5707963 0 0
- joint Roller_81_94_joint: mimic joint=Roller_81_81_joint multiplier=1 offset=0 -> (none); origin xyz=-8.905875 0 0.15 rpy=1.5707963 0 0 -> xyz=-8.905875 0 1.15 rpy=1.5707963 0 0
- joint Roller_81_95_joint: mimic joint=Roller_81_81_joint multiplier=1 offset=0 -> (none); origin xyz=-9.001125 0 0.15 rpy=1.5707963 0 0 -> xyz=-9.001125 0 1.15 rpy=1.5707963 0 0
- joint Roller_81_96_joint: mimic joint=Roller_81_81_joint multiplier=1 offset=0 -> (none); origin xyz=-9.096375 0 0.15 rpy=1.5707963 0 0 -> xyz=-9.096375 0 1.15 rpy=1.5707963 0 0
- joint Roller_97_100_joint: mimic joint=Roller_97_97_joint multiplier=1 offset=0 -> (none); origin xyz=-9.477375 0 0.15 rpy=1.5707963 0 0 -> xyz=-9.477375 0 1.15 rpy=1.5707963 0 0
- joint Roller_97_101_joint: mimic joint=Roller_97_97_joint multiplier=1 offset=0 -> (none); origin xyz=-9.572625 0 0.15 rpy=1.5707963 0 0 -> xyz=-9.572625 0 1.15 rpy=1.5707963 0 0
- joint Roller_97_102_joint: mimic joint=Roller_97_97_joint multiplier=1 offset=0 -> (none); origin xyz=-9.667875 0 0.15 rpy=1.5707963 0 0 -> xyz=-9.667875 0 1.15 rpy=1.5707963 0 0
- joint Roller_97_103_joint: mimic joint=Roller_97_97_joint multiplier=1 offset=0 -> (none); origin xyz=-9.763125 0 0.15 rpy=1.5707963 0 0 -> xyz=-9.763125 0 1.15 rpy=1.5707963 0 0
- joint Roller_97_104_joint: mimic joint=Roller_97_97_joint multiplier=1 offset=0 -> (none); origin xyz=-9.858375 0 0.15 rpy=1.5707963 0 0 -> xyz=-9.858375 0 1.15 rpy=1.5707963 0 0
- joint Roller_97_105_joint: mimic joint=Roller_97_97_joint multiplier=1 offset=0 -> (none); origin xyz=-9.953625 0 0.15 rpy=1.5707963 0 0 -> xyz=-9.953625 0 1.15 rpy=1.5707963 0 0
- joint Roller_97_106_joint: mimic joint=Roller_97_97_joint multiplier=1 offset=0 -> (none); origin xyz=-10.048875 0 0.15 rpy=1.5707963 0 0 -> xyz=-10.048875 0 1.15 rpy=1.5707963 0 0
- joint Roller_97_107_joint: mimic joint=Roller_97_97_joint multiplier=1 offset=0 -> (none); origin xyz=-10.144125 0 0.15 rpy=1.5707963 0 0 -> xyz=-10.144125 0 1.15 rpy=1.5707963 0 0
- joint Roller_97_108_joint: mimic joint=Roller_97_97_joint multiplier=1 offset=0 -> (none); origin xyz=-10.239375 0 0.15 rpy=1.5707963 0 0 -> xyz=-10.239375 0 1.15 rpy=1.5707963 0 0
- joint Roller_97_109_joint: mimic joint=Roller_97_97_joint multiplier=1 offset=0 -> (none); origin xyz=-10.334625 0 0.15 rpy=1.5707963 0 0 -> xyz=-10.334625 0 1.15 rpy=1.5707963 0 0
- joint Roller_97_110_joint: mimic joint=Roller_97_97_joint multiplier=1 offset=0 -> (none); origin xyz=-10.429875000000001 0 0.15 rpy=1.5707963 0 0 -> xyz=-10.429875000000001 0 1.15 rpy=1.5707963 0 0
- joint Roller_97_111_joint: mimic joint=Roller_97_97_joint multiplier=1 offset=0 -> (none); origin xyz=-10.525125000000001 0 0.15 rpy=1.5707963 0 0 -> xyz=-10.525125000000001 0 1.15 rpy=1.5707963 0 0
- joint Roller_97_112_joint: mimic joint=Roller_97_97_joint multiplier=1 offset=0 -> (none); origin xyz=-10.620375000000001 0 0.15 rpy=1.5707963 0 0 -> xyz=-10.620375000000001 0 1.15 rpy=1.5707963 0 0
- joint Roller_97_97_joint: origin xyz=-9.191625 0 0.15 rpy=1.570796 0 0 -> xyz=-9.191625 0 1.15 rpy=1.570796 0 0
- joint Roller_97_98_joint: mimic joint=Roller_97_97_joint multiplier=1 offset=0 -> (none); origin xyz=-9.286875 0 0.15 rpy=1.5707963 0 0 -> xyz=-9.286875 0 1.15 rpy=1.5707963 0 0
- joint Roller_97_99_joint: mimic joint=Roller_97_97_joint multiplier=1 offset=0 -> (none); origin xyz=-9.382125 0 0.15 rpy=1.5707963 0 0 -> xyz=-9.382125 0 1.15 rpy=1.5707963 0 0
