Commit message: add bunch of stuff

File: custom40ftStraight_v3.xacro (robot description, xacro)
@@ -21,5 +21,5 @@
             <origin xyz="-6.096 0 0" rpy="0 0 0" />
             <geometry>
-                <box size="12.192 1.219 0.1"/>
+                <box size="12.192 1.219 2.0"/>
             </geometry>
             <material name="gray">
@@ -28,11 +28,11 @@
         </visual>
         <collision>
-            <origin xyz="-6.096 0 0" rpy="0 0 0" />
-            <geometry>
-                <box size="12.192 1.219 0.1"/>
-            </geometry>
-        </collision>
-        <inertial>
-            <origin xyz="-6.096 0 0" rpy="0 0 0" />
+            <origin xyz="-6.096 0 1.0" rpy="0 0 0" />
+            <geometry>
+                <box size="12.192 1.219 2.0"/>
+            </geometry>
+        </collision>
+        <inertial>
+            <origin xyz="-6.096 0 1.0" rpy="0 0 0" />
             <mass value="20.0"/>
             <inertia ixx="0.2" iyy="0.2" izz="0.2"/>
@@ -42,7 +42,7 @@
     <link name="leftFrame">
         <visual>
-            <origin xyz="-6.096 0 0" rpy="0 0 0" />
-            <geometry>
-                <box size="12.192 0.05 0.5"/>
+            <origin xyz="-6.096 0 0.0" rpy="0 0 0" />
+            <geometry>
+                <box size="12.192 0.05 2.5"/>
             </geometry>
             <material name="gray">
@@ -51,11 +51,11 @@
         </visual>
         <collision>
-            <origin xyz="-6.096 0 0" rpy="0 0 0" />
-            <geometry>
-                <box size="12.192 0.05 0.5"/>
-            </geometry>
-        </collision>
-        <inertial>
-            <origin xyz="-6.096 0 0" rpy="0 0 0" />
+            <origin xyz="-6.096 0 0.0" rpy="0 0 0" />
+            <geometry>
+                <box size="12.192 0.05 2.5"/>
+            </geometry>
+        </collision>
+        <inertial>
+            <origin xyz="-6.096 0 0.0" rpy="0 0 0" />
             <mass value="20.0"/>
             <inertia ixx="0.2" iyy="0.2" izz="0.2"/>
@@ -73,5 +73,5 @@
             <origin xyz="-6.096 0 0" rpy="0 0 0" />
             <geometry>
-                <box size="12.192 0.05 0.5"/>
+                <box size="12.192 0.05 2.5"/>
             </geometry>
             <material name="gray">
@@ -82,5 +82,5 @@
             <origin xyz="-6.096 0 0" rpy="0 0 0" />
             <geometry>
-                <box size="12.192 0.05 0.5"/>
+                <box size="12.192 0.05 2.5"/>
             </geometry>
         </collision>
@@ -122,5 +122,5 @@
         <parent link="base_link"/>
         <child link="Roller_1"/>
-        <origin xyz="-${roller_pitch/2} 0 0.15" rpy="1.570796 0 0"/>
+        <origin xyz="-${roller_pitch/2} 0 1.15" rpy="1.570796 0 0"/>
         <axis xyz="0 0 1"/>
         <dynamics damping="1.0" friction="0.0"/>
@@ -150,5 +150,5 @@
             <parent link="base_link"/>
             <child link="Roller_${rollerNum}"/>
-            <origin xyz="-${(rollerNum-1)*roller_pitch + roller_pitch/2} 0 0.15" rpy="${pi/2} 0 0"/>
+            <origin xyz="-${(rollerNum-1)*roller_pitch + roller_pitch/2} 0 1.15" rpy="${pi/2} 0 0"/>
             <axis xyz="0 0 1"/>
             <dynamics damping="1.0" friction="0.0"/>
@@ -179,5 +179,5 @@
         <parent link="base_link"/>
         <child link="Roller_17"/>
-        <origin xyz="-${(17-1)*roller_pitch + roller_pitch/2} 0 0.15" rpy="1.570796 0 0"/>
+        <origin xyz="-${(17-1)*roller_pitch + roller_pitch/2} 0 1.15" rpy="1.570796 0 0"/>
         <axis xyz="0 0 1"/>
         <dynamics damping="1.0" friction="0.0"/>
@@ -207,5 +207,5 @@
             <parent link="base_link"/>
             <child link="Roller_${rollerNum}"/>
-            <origin xyz="-${(rollerNum-1)*roller_pitch + roller_pitch/2} 0 0.15" rpy="${pi/2} 0 0"/>
+            <origin xyz="-${(rollerNum-1)*roller_pitch + roller_pitch/2} 0 1.15" rpy="${pi/2} 0 0"/>
             <axis xyz="0 0 1"/>
             <dynamics damping="1.0" friction="0.0"/>
@@ -237,5 +237,5 @@
         <parent link="base_link"/>
         <child link="Roller_33"/>
-        <origin xyz="-${(32)*roller_pitch + roller_pitch/2} 0 0.15" rpy="1.570796 0 0"/>
+        <origin xyz="-${(32)*roller_pitch + roller_pitch/2} 0 1.15" rpy="1.570796 0 0"/>
         <axis xyz="0 0 1"/>
         <dynamics damping="1.0" friction="0.0"/>
@@ -265,5 +265,5 @@
             <parent link="base_link"/>
             <child link="Roller_${rollerNum}"/>
-            <origin xyz="-${(rollerNum-1)*roller_pitch + roller_pitch/2} 0 0.15" rpy="${pi/2} 0 0"/>
+            <origin xyz="-${(rollerNum-1)*roller_pitch + roller_pitch/2} 0 1.15" rpy="${pi/2} 0 0"/>
             <axis xyz="0 0 1"/>
             <dynamics damping="1.0" friction="0.0"/>
@@ -294,5 +294,5 @@
         <parent link="base_link"/>
         <child link="Roller_49"/>
-        <origin xyz="-${(49-1)*roller_pitch + roller_pitch/2} 0 0.15" rpy="1.570796 0 0"/>
+        <origin xyz="-${(49-1)*roller_pitch + roller_pitch/2} 0 1.15" rpy="1.570796 0 0"/>
         <axis xyz="0 0 1"/>
         <dynamics damping="1.0" friction="0.0"/>
@@ -322,5 +322,5 @@
             <parent link="base_link"/>
             <child link="Roller_${rollerNum}"/>
-            <origin xyz="-${(rollerNum-1)*roller_pitch + roller_pitch/2} 0 0.15" rpy="${pi/2} 0 0"/>
+            <origin xyz="-${(rollerNum-1)*roller_pitch + roller_pitch/2} 0 1.15" rpy="${pi/2} 0 0"/>
             <axis xyz="0 0 1"/>
             <dynamics damping="1.0" friction="0.0"/>
@@ -352,5 +352,5 @@
         <parent link="base_link"/>
         <child link="Roller_65"/>
-        <origin xyz="-${(64)*roller_pitch + roller_pitch/2} 0 0.15" rpy="1.570796 0 0"/>
+        <origin xyz="-${(64)*roller_pitch + roller_pitch/2} 0 1.15" rpy="1.570796 0 0"/>
         <axis xyz="0 0 1"/>
         <dynamics damping="1.0" friction="0.0"/>
@@ -380,5 +380,5 @@
             <parent link="base_link"/>
             <child link="Roller_${rollerNum}"/>
-            <origin xyz="-${(rollerNum-1)*roller_pitch + roller_pitch/2} 0 0.15" rpy="${pi/2} 0 0"/>
+            <origin xyz="-${(rollerNum-1)*roller_pitch + roller_pitch/2} 0 1.15" rpy="${pi/2} 0 0"/>
             <axis xyz="0 0 1"/>
             <dynamics damping="1.0" friction="0.0"/>
@@ -409,5 +409,5 @@
         <parent link="base_link"/>
         <child link="Roller_81"/>
-        <origin xyz="-${(81-1)*roller_pitch + roller_pitch/2} 0 0.15" rpy="1.570796 0 0"/>
+        <origin xyz="-${(81-1)*roller_pitch + roller_pitch/2} 0 1.15" rpy="1.570796 0 0"/>
         <axis xyz="0 0 1"/>
         <dynamics damping="1.0" friction="0.0"/>
@@ -437,5 +437,5 @@
             <parent link="base_link"/>
             <child link="Roller_${rollerNum}"/>
-            <origin xyz="-${(rollerNum-1)*roller_pitch + roller_pitch/2} 0 0.15" rpy="${pi/2} 0 0"/>
+            <origin xyz="-${(rollerNum-1)*roller_pitch + roller_pitch/2} 0 1.15" rpy="${pi/2} 0 0"/>
             <axis xyz="0 0 1"/>
             <dynamics damping="1.0" friction="0.0"/>
@@ -467,5 +467,5 @@
         <parent link="base_link"/>
         <child link="Roller_97"/>
-        <origin xyz="-${(96)*roller_pitch + roller_pitch/2} 0 0.15" rpy="1.570796 0 0"/>
+        <origin xyz="-${(96)*roller_pitch + roller_pitch/2} 0 1.15" rpy="1.570796 0 0"/>
         <axis xyz="0 0 1"/>
         <dynamics damping="1.0" friction="0.0"/>
@@ -495,5 +495,5 @@
             <parent link="base_link"/>
             <child link="Roller_${rollerNum}"/>
-            <origin xyz="-${(rollerNum-1)*roller_pitch + roller_pitch/2} 0 0.15" rpy="${pi/2} 0 0"/>
+            <origin xyz="-${(rollerNum-1)*roller_pitch + roller_pitch/2} 0 1.15" rpy="${pi/2} 0 0"/>
             <axis xyz="0 0 1"/>
             <dynamics damping="1.0" friction="0.0"/>
@@ -524,5 +524,5 @@
         <parent link="base_link"/>
         <child link="Roller_113"/>
-        <origin xyz="-${(113-1)*roller_pitch + roller_pitch/2} 0 0.15" rpy="1.570796 0 0"/>
+        <origin xyz="-${(113-1)*roller_pitch + roller_pitch/2} 0 1.15" rpy="1.570796 0 0"/>
         <axis xyz="0 0 1"/>
         <dynamics damping="1.0" friction="0.0"/>
@@ -552,5 +552,5 @@
             <parent link="base_link"/>
             <child link="Roller_${rollerNum}"/>
-            <origin xyz="-${(rollerNum-1)*roller_pitch + roller_pitch/2} 0 0.15" rpy="${pi/2} 0 0"/>
+            <origin xyz="-${(rollerNum-1)*roller_pitch + roller_pitch/2} 0 1.15" rpy="${pi/2} 0 0"/>
             <axis xyz="0 0 1"/>
             <dynamics damping="1.0" friction="0.0"/>

Commit message: exclude mimics

File: custom40ftStraight_v3.xacro (robot description, xacro)
@@ -153,5 +153,4 @@
             <axis xyz="0 0 1"/>
             <dynamics damping="1.0" friction="0.0"/>
-            <mimic joint="Roller_1_1_joint" multiplier="1" offset="0" />
         </joint>
     </xacro:macro>
@@ -210,5 +209,4 @@
             <axis xyz="0 0 1"/>
             <dynamics damping="1.0" friction="0.0"/>
-            <mimic joint="Roller_17_17_joint" multiplier="1" offset="0" />
         </joint>
     </xacro:macro>
@@ -268,5 +266,4 @@
             <axis xyz="0 0 1"/>
             <dynamics damping="1.0" friction="0.0"/>
-            <mimic joint="Roller_33_33_joint" multiplier="1" offset="0" />
         </joint>
     </xacro:macro>
@@ -325,5 +322,4 @@
             <axis xyz="0 0 1"/>
             <dynamics damping="1.0" friction="0.0"/>
-            <mimic joint="Roller_49_49_joint" multiplier="1" offset="0" />
         </joint>
     </xacro:macro>
@@ -383,5 +379,4 @@
             <axis xyz="0 0 1"/>
             <dynamics damping="1.0" friction="0.0"/>
-            <mimic joint="Roller_65_65_joint" multiplier="1" offset="0" />
         </joint>
     </xacro:macro>
@@ -440,5 +435,4 @@
             <axis xyz="0 0 1"/>
             <dynamics damping="1.0" friction="0.0"/>
-            <mimic joint="Roller_81_81_joint" multiplier="1" offset="0" />
         </joint>
     </xacro:macro>
@@ -498,5 +492,4 @@
             <axis xyz="0 0 1"/>
             <dynamics damping="1.0" friction="0.0"/>
-            <mimic joint="Roller_97_97_joint" multiplier="1" offset="0" />
         </joint>
     </xacro:macro>
@@ -555,5 +548,4 @@
             <axis xyz="0 0 1"/>
             <dynamics damping="1.0" friction="0.0"/>
-            <mimic joint="Roller_113_113_joint" multiplier="1" offset="0" />
         </joint>
     </xacro:macro>

Commit message: did not use BaseBox anymore

File: custom40ftStraight_v3.xacro (robot description, xacro)
@@ -28,5 +28,5 @@
         </visual>
         <collision>
-            <origin xyz="-6.096 0 1.0" rpy="0 0 0" />
+            <origin xyz="-6.096 0 0.0" rpy="0 0 0" />
             <geometry>
                 <box size="12.192 1.219 2.0"/>
